File: am_receiver_v2.kicad_sch (KiCad schematic)
At the start: 4 parts

Commit message: added description
Other:
- note added: "ŁK 2025"
Changed lines of the file:
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@@
+		)
+	)
+	(text "ŁK 2025"
+		(exclude_from_sim no)
+		(at 273.812 189.992 0)
+		(effects
+			(font
+				(size 2.032 2.032)
+			)
 		)
 	)
